File: hw/sch_pcb/TFGPS01B.kicad_pcb (KiCad board)
At the start: 4 copper layers, 51 x 51 mm, 72 parts, among them J1 SM10B-GHS-TB, J2 USBC_USB4105-GF-A, J3 SM06B-GHS-TB, J4 SM04B-GHS-TB, J5 SM08B-GHS-TB, M1 HOLE, M2 HOLE, M3 HOLE, M4 HOLE, Q1 BC817-25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

Commit message: Edit schema
Parts:
- removed G***: LOGO, MLAB_LOGA:TF
- added R25: 10k, Mlab_R:SMD-0805, F.Cu at (63.4, -10.4)
- C13: value 1pF -> 1p5F
- L2: value 4n7H -> 5n6H
- R13: value 100R -> 10k
- R28: value 100R -> 20k
- U4: value MAX2656 -> MAX2655
Connections:
- J2 pad A8: (no net) -> unconnected-(J2-PadA8)
- J2 pad B8: (no net) -> unconnected-(J2-PadB8)
- U1 pad 4: (no net) -> unconnected-(U1-Pad4)
- U3 pad 1: (no net) -> unconnected-(U3-Pad1)
- U3 pad 14: (no net) -> unconnected-(U3-Pad14)
- U3 pad 17: (no net) -> unconnected-(U3-Pad17)
- U3 pad 2: (no net) -> unconnected-(U3-Pad2)
- U3 pad 8: (no net) -> unconnected-(U3-Pad8)

Commit message: Edit schema
Parts:
- added D9: 15MQ040N, Diode_SMD:D_SMA, F.Cu at (62.5, -6.35)
- added F1: 750mA, Fuse:Fuse_0805_2012Metric, F.Cu at (60.7, -2.60)
Connections:
- J2 pad A4/B9: +5V -> /VBUS
- J2 pad B4/A9: +5V -> /VBUS
- U2 pad 5: +5V -> /VBUS
Changed lines of the file:
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@@
   (net 64 "unconnected-(U3-Pad14)")
   (net 65 "unconnected-(U3-Pad17)")
+  (net 66 "Net-(D9-Pad2)")
+  (net 67 "/VBUS")
   (footprint "Mlab_Mechanical:MountingHole_3mm" placed (layer "F.Cu")
     (at 45.42 -5.38)
@@
       (net 1 "GND") (pintype "input") (clearance 1) (zone_connect 2))
     (model "${MLAB}/src/3d/mechanical/m3_komplet.step"
+      (offset (xyz 0 0 0))
+      (scale (xyz 1 1 1))
+      (rotate (xyz 0 0 0))
+    )
+  )
+  (footprint "Fuse:Fuse_0805_2012Metric" (layer "F.Cu")
+    (at 60.664 -2.6)
+    (descr "Fuse SMD 0805 (2012 Metric), square (rectangular) end terminal, IPC_7351 nominal, (Body size source: https://docs.google.com/spreadsheets/d/1BsfQQcO9C6DZCsRaXUlFlo91Tg2WpOkGARC1WS5S8t0/edit?usp=sharing), generated with kicad-footprint-generator")
+    (tags "fuse")
+    (property "Sheetfile" "TFGPS01B.kicad_sch")
+    (property "Sheetname" "")
+    (attr smd)
+    (fp_text reference "F1" (at 0 -1.65) (layer "F.SilkS")
+      (effects (font (size 1 1) (thickness 0.15)))
+    )
+    (fp_text value "750mA" (at 0 1.65) (layer "F.Fab")
+      (effects (font (size 1 1) (thickness 0.15)))
+    )
+    (fp_text user "${REFERENCE}" (at 0 0) (layer "F.Fab")
+      (effects (font (size 0.5 0.5) (thickness 0.08)))
+    )
+    (fp_line (start -0.258578 0.71) (end 0.258578 0.71) (layer "F.SilkS") (width 0.12))
+    (fp_line (start -0.258578 -0.71) (end 0.258578 -0.71) (layer "F.SilkS") (width 0.12))
+    (fp_line (start 1.68 -0.95) (end 1.68 0.95) (layer "F.CrtYd") (width 0.05))
+    (fp_line (start 1.68 0.95) (end -1.68 0.95) (layer "F.CrtYd") (width 0.05))
+    (fp_line (start -1.68 0.95) (end -1.68 -0.95) (layer "F.CrtYd") (width 0.05))
+    (fp_line (start -1.68 -0.95) (end 1.68 -0.95) (layer "F.CrtYd") (width 0.05))
+    (fp_line (start 1 -0.6) (end 1 0.6) (layer "F.Fab") (width 0.1))
+    (fp_line (start 1 0.6) (end -1 0.6) (layer "F.Fab") (width 0.1))
+    (fp_line (start -1 -0.6) (end 1 -0.6) (layer "F.Fab") (width 0.1))
+    (fp_line (start -1 0.6) (end -1 -0.6) (layer "F.Fab") (width 0.1))
+    (pad "1" smd roundrect locked (at -0.9375 0) (size 0.975 1.4) (layers "F.Cu" "F.Paste" "F.Mask") (roundrect_rratio 0.25)
+      (net 67 "/VBUS") (pintype "passive"))
+    (pad "2" smd roundrect locked (at 0.9375 0) (size 0.975 1.4) (layers "F.Cu" "F.Paste" "F.Mask") (roundrect_rratio 0.25)
+      (net 66 "Net-(D9-Pad2)") (pintype "passive"))
+    (model "${KISYS3DMOD}/Fuse.3dshapes/Fuse_0805_2012Metric.wrl"
       (offset (xyz 0 0 0))
       (scale (xyz 1 1 1))
@@
       (net 57 "/SAFE_VCC") (pintype "passive"))
     (model "${KISYS3DMOD}/Resistor_SMD.3dshapes/R_0805_2012Metric.wrl"
+      (offset (xyz 0 0 0))
+      (scale (xyz 1 1 1))
+      (rotate (xyz 0 0 0))
+    )
+  )
+  (footprint "Diode_SMD:D_SMA" (layer "F.Cu")
+    (at 62.484 -6.35)
+    (descr "Diode SMA (DO-214AC)")
+    (tags "Diode SMA (DO-214AC)")
+    (property "Sheetfile" "TFGPS01B.kicad_sch")
+    (property "Sheetname" "")
+    (property "UST_ID" "5c70984512875079b91f88b0")
+    (attr smd)
+    (fp_text reference "D9" (at 0 -2.5) (layer "F.SilkS")
+      (effects (font (size 1 1) (thickness 0.15)))
+    )
+    (fp_text value "15MQ040N" (at 0 2.6) (layer "F.Fab")
+      (effects (font (size 1 1) (thickness 0.15)))
+    )
+    (fp_text user "${REFERENCE}" (at 0 -2.5) (layer "F.Fab")
+      (effects (font (size 1 1) (thickness 0.15)))
+    )
+    (fp_line (start -3.4 1.65) (end 2 1.65) (layer "F.SilkS") (width 0.12))
+    (fp_line (start -3.4 -1.65) (end -3.4 1.65) (layer "F.SilkS") (width 0.12))
+    (fp_line (start -3.4 -1.65) (end 2 -1.65) (layer "F.SilkS") (width 0.12))
+    (fp_line (start -3.5 -1.75) (end 3.5 -1.75) (layer "F.CrtYd") (width 0.05))
+    (fp_line (start -3.5 1.75) (end -3.5 -1.75) (layer "F.CrtYd") (width 0.05))
+    (fp_line (start 3.5 1.75) (end -3.5 1.75) (layer "F.CrtYd") (width 0.05))
+    (fp_line (start 3.5 -1.75) (end 3.5 1.75) (layer "F.CrtYd") (width 0.05))
+    (fp_line (start 2.3 1.5) (end -2.3 1.5) (layer "F.Fab") (width 0.1))
+    (fp_line (start 0.50118 0.00102) (end 1.4994 0.00102) (layer "F.Fab") (width 0.1))
+    (fp_line (start 2.3 -1.5) (end -2.3 -1.5) (layer "F.Fab") (width 0.1))
+    (fp_line (start -2.3 1.5) (end -2.3 -1.5) (layer "F.Fab") (width 0.1))
+    (fp_line (start -0.64944 0.00102) (end 0.50118 0.75032) (layer "F.Fab") (width 0.1))
+    (fp_line (start -0.64944 0.00102) (end 0.50118 -0.79908) (layer "F.Fab") (width 0.1))
+    (fp_line (start -0.64944 0.00102) (end -1.55114 0.00102) (layer "F.Fab") (width 0.1))
+    (fp_line (start 2.3 -1.5) (end 2.3 1.5) (layer "F.Fab") (width 0.1))
+    (fp_line (start 0.50118 0.75032) (end 0.50118 -0.79908) (layer "F.Fab") (width 0.1))
+    (fp_line (start -0.64944 -0.79908) (end -0.64944 0.80112) (layer "F.Fab") (width 0.1))
+    (pad "1" smd rect locked (at -2 0) (size 2.5 1.8) (layers "F.Cu" "F.Paste" "F.Mask")
+      (net 7 "+5V") (pinfunction "K") (pintype "passive"))
+    (pad "2" smd rect locked (at 2 0) (size 2.5 1.8) (layers "F.Cu" "F.Paste" "F.Mask")
+      (net 66 "Net-(D9-Pad2)") (pinfunction "A") (pintype "passive"))
+    (model "${KISYS3DMOD}/Diode_SMD.3dshapes/D_SMA.wrl"
       (offset (xyz 0 0 0))
       (scale (xyz 1 1 1))
@@
       (net 12 "/D-") (pinfunction "IO2") (pintype "passive"))
     (pad "5" smd rect locked (at 1.1 0 180) (size 1.06 0.65) (layers "B.Cu" "B.Paste" "B.Mask")
-      (net 7 "+5V") (pinfunction "VBUS") (pintype "passive"))
+      (net 67 "/VBUS") (pinfunction "VBUS") (pintype "passive"))
     (pad "6" smd rect locked (at 1.1 0.95 180) (size 1.06 0.65) (layers "B.Cu" "B.Paste" "B.Mask")
       (net 11 "/D+") (pinfunction "IO1") (pintype "passive"))
@@
       (net 1 "GND") (pinfunction "GND") (pintype "passive"))
     (pad "A4/B9" smd rect locked (at -2.4 4.755 90) (size 0.6 1.15) (layers "B.Cu" "B.Paste" "B.Mask")
-      (net 7 "+5V") (pinfunction "VBUS") (pintype "passive"))
+      (net 67 "/VBUS") (pinfunction "VBUS") (pintype "passive"))
     (pad "A5" smd rect locked (at -1.25 4.755 90) (size 0.3 1.15) (layers "B.Cu" "B.Paste" "B.Mask")
       (net 40 "Net-(J2-PadA5)") (pinfunction "CC1") (pintype "bidirectional"))
@@
       (net 1 "GND") (pinfunction "GND") (pintype "passive"))
     (pad "B4/A9" smd rect locked (at 2.4 4.755 90) (size 0.6 1.15) (layers "B.Cu" "B.Paste" "B.Mask")
-      (net 7 "+5V") (pinfunction "VBUS") (pintype "passive"))
+      (net 67 "/VBUS") (pinfunction "VBUS") (pintype "passive"))
     (pad "B5" smd rect locked (at 1.75 4.755 90) (size 0.3 1.15) (layers "B.Cu" "B.Paste" "B.Mask")
       (net 41 "Net-(J2-PadB5)") (pinfunction "CC2") (pintype "bidirectional"))

Commit message: Edit SCH
Parts:
- removed F1: 750mA, Fuse:Fuse_0805_2012Metric
- D9: value 15MQ040N -> BZX585-B5V6.115; footprint Diode_SMD:D_SMA -> Diode_SMD:D_SOD-523; moved to B.Cu
- R25: moved to B.Cu
- moved D9 63.8 mm to (9.40, -41.8), turned to 90 degrees
- moved R25 47.2 mm to (28.4, -42.1), turned to 90 degrees
Connections:
- D9 pad 1: +5V -> /VBUS
- D9 pad 2: Net-(D9-Pad2) -> +5V
- L1 pad 1: +5V -> /VBUS
Routing:
- net +5V: track 152.5 -> 123.1 mm, vias 9 -> 6
- net /VBUS: track 0.00 -> 19.3 mm, vias 0 -> 3
- net /SAFETY_SW_LED: track 74.8 -> 80.6 mm
- net /SAFE_VCC: track 77.1 -> 79.3 mm
Other:
- board text added: "TFGPS01B JACHO 2021"
- board text removed: "TFGPS01A JACHO 2020"

Commit message: Edit PCB
Parts:
- added D10: BZX585-B5V6.115, Diode_SMD:D_SOD-523, B.Cu at (9.40, -39.9)
- moved D9 1.05 mm to (9.65, -42.8)
Connections:
- D9 pad 1: /VBUS -> Net-(D9-Pad1)
- L1 pad 1: /VBUS -> Net-(D9-Pad1)
Routing:
- net Net-(D9-Pad1): track 0.00 -> 12.0 mm, vias 0 -> 2
- net /VBUS: track 19.3 -> 17.4 mm
- net +5V: track 123.1 -> 122.0 mm
Changed lines of the file:
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@@
   (net 65 "unconnected-(U3-Pad17)")
   (net 66 "/VBUS")
+  (net 67 "Net-(D9-Pad1)")
   (footprint "Mlab_Mechanical:MountingHole_3mm" placed (layer "F.Cu")
     (at 45.42 -5.38)
@@
     (property "UST_ID" "5c70984512875079b91f88b3")
     (attr smd)
-    (fp_text reference "D1" (at 2.06 2.159 90) (layer "B.SilkS")
+    (fp_text reference "D1" (at -0.152 -0.051 90) (layer "B.SilkS")
       (effects (font (size 1 1) (thickness 0.15)) (justify mirror))
     )
@@
   )
   (footprint "Diode_SMD:D_SOD-523" (layer "B.Cu")
-    (at 9.398 -41.783 90)
+    (at 9.652 -42.799 90)
     (descr "http://www.diodes.com/datasheets/ap02001.pdf p.144")
     (tags "Diode SOD523")
@@
     (property "UST_id" "")
     (attr smd)
-    (fp_text reference "D9" (at 0 -1.524 90) (layer "B.SilkS")
+    (fp_text reference "D9" (at 0 -1.524 90) (layer "B.SilkS") hide
       (effects (font (size 1 1) (thickness 0.15)) (justify mirror))
     )
@@
     (fp_line (start -0.65 0.45) (end 0.65 0.45) (layer "B.Fab") (width 0.1))
     (pad "1" smd rect locked (at -0.7 0 270) (size 0.6 0.7) (layers "B.Cu" "B.Paste" "B.Mask")
-      (net 66 "/VBUS") (pinfunction "K") (pintype "passive"))
+      (net 67 "Net-(D9-Pad1)") (pinfunction "K") (pintype "passive"))
     (pad "2" smd rect locked (at 0.7 0 270) (size 0.6 0.7) (layers "B.Cu" "B.Paste" "B.Mask")
       (net 7 "+5V") (pinfunction "A") (pintype "passive"))
@@
     )
   )
+  (footprint "Diode_SMD:D_SOD-523" (layer "B.Cu")
+    (at 9.398 -39.878 -90)
+    (descr "http://www.diodes.com/datasheets/ap02001.pdf p.144")
+    (tags "Diode SOD523")
+    (property "Sheetfile" "TFGPS01B.kicad_sch")
+    (property "Sheetname" "")
+    (property "UST_ID" "60879d38128750769ee58e48")
+    (property "UST_id" "")
+    (attr smd)
+    (fp_text reference "D10" (at 0 1.3 90) (layer "B.SilkS") hide
+      (effects (font (size 1 1) (thickness 0.15)) (justify mirror))
+    )
+    (fp_text value "BZX585-B5V6.115" (at 0 -1.4 90) (layer "B.Fab") hide
+      (effects (font (size 1 1) (thickness 0.15)) (justify mirror))
+    )
+    (fp_text user "${REFERENCE}" (at 0 1.3 90) (layer "B.Fab")
+      (effects (font (size 1 1) (thickness 0.15)) (justify mirror))
+    )
+    (fp_line (start -1.15 0.6) (end -1.15 -0.6) (layer "B.SilkS") (width 0.12))
+    (fp_line (start 0.7 -0.6) (end -1.15 -0.6) (layer "B.SilkS") (width 0.12))
+    (fp_line (start 0.7 0.6) (end -1.15 0.6) (layer "B.SilkS") (width 0.12))
+    (fp_line (start 1.25 -0.7) (end -1.25 -0.7) (layer "B.CrtYd") (width 0.05))
+    (fp_line (start 1.25 0.7) (end 1.25 -0.7) (layer "B.CrtYd") (width 0.05))
+    (fp_line (start -1.25 -0.7) (end -1.25 0.7) (layer "B.CrtYd") (width 0.05))
+    (fp_line (start -1.25 0.7) (end 1.25 0.7) (layer "B.CrtYd") (width 0.05))
+    (fp_line (start 0.65 0.45) (end 0.65 -0.45) (layer "B.Fab") (width 0.1))
+    (fp_line (start -0.2 0) (end -0.35 0) (layer "B.Fab") (width 0.1))
+    (fp_line (start -0.65 0.45) (end 0.65 0.45) (layer "B.Fab") (width 0.1))
+    (fp_line (start -0.2 0) (end 0.1 -0.2) (layer "B.Fab") (width 0.1))
+    (fp_line (start 0.1 -0.2) (end 0.1 0.2) (layer "B.Fab") (width 0.1))
+    (fp_line (start 0.1 0) (end 0.25 0) (layer "B.Fab") (width 0.1))
+    (fp_line (start 0.65 -0.45) (end -0.65 -0.45) (layer "B.Fab") (width 0.1))
+    (fp_line (start -0.65 -0.45) (end -0.65 0.45) (layer "B.Fab") (width 0.1))
+    (fp_line (start 0.1 0.2) (end -0.2 0) (layer "B.Fab") (width 0.1))
+    (fp_line (start -0.2 -0.2) (end -0.2 0.2) (layer "B.Fab") (width 0.1))
+    (pad "1" smd rect locked (at -0.7 0 90) (size 0.6 0.7) (layers "B.Cu" "B.Paste" "B.Mask")
+      (net 67 "Net-(D9-Pad1)") (pinfunction "K") (pintype "passive"))
+    (pad "2" smd rect locked (at 0.7 0 90) (size 0.6 0.7) (layers "B.Cu" "B.Paste" "B.Mask")
+      (net 66 "/VBUS") (pinfunction "A") (pintype "passive"))
+    (model "${KISYS3DMOD}/Diode_SMD.3dshapes/D_SOD-523.wrl"
+      (offset (xyz 0 0 0))
+      (scale (xyz 1 1 1))
+      (rotate (xyz 0 0 0))
+    )
+  )
   (footprint "Mlab_R:SMD-0805" (layer "B.Cu")
     (at 3.2385 -25.527 180)
@@
     (fp_line (start 1.6 1.25) (end 1.6 -1.25) (layer "B.Fab") (width 0.1))
     (pad "1" smd roundrect locked (at -1.4 0) (size 1.25 2.65) (layers "B.Cu" "B.Paste" "B.Mask") (roundrect_rratio 0.2)
-      (net 66 "/VBUS") (pinfunction "1") (pintype "passive"))
+      (net 67 "Net-(D9-Pad1)") (pinfunction "1") (pintype "passive"))
     (pad "2" smd roundrect locked (at 1.4 0) (size 1.25 2.65) (layers "B.Cu" "B.Paste" "B.Mask") (roundrect_rratio 0.2)
       (net 9 "Net-(C3-Pad1)") (pinfunction "2") (pintype "passive"))
@@
   (via (at 49.614001 -34.967999) (size 0.7) (drill 0.3) (layers "F.Cu" "B.Cu") (net 7))
   (via (at 29.464 -4.572) (size 0.8) (drill 0.4) (layers "F.Cu" "B.Cu") (net 7))
-  (via (at 9.652 -43.688) (size 0.7) (drill 0.3) (layers "F.Cu" "B.Cu") (net 7))
+  (via (at 9.906 -44.577) (size 0.7) (drill 0.3) (layers "F.Cu" "B.Cu") (net 7))
   (via (at 46.228 -13.97) (size 0.8) (drill 0.4) (layers "F.Cu" "B.Cu") (net 7))
   (via (at 38.9255 -44.6405) (size 0.7) (drill 0.3) (layers "F.Cu" "B.Cu") (net 7))
   (segment (start 46.228 -13.97) (end 36.83 -4.572) (width 1) (layer "In2.Cu") (net 7))
-  (segment (start 9.906 -43.942) (end 9.652 -43.688) (width 1) (layer "In2.Cu") (net 7))
   (segment (start 49.614001 -39.793999) (end 49.614001 -34.967999) (width 1) (layer "In2.Cu") (net 7))
-  (segment (start 9.906 -45.466) (end 9.906 -43.942) (width 1) (layer "In2.Cu") (net 7))
+  (segment (start 9.906 -45.466) (end 9.906 -44.577) (width 1) (layer "In2.Cu") (net 7))
   (segment (start 12.446 -48.006) (end 30.48 -48.006) (width 1) (layer "In2.Cu") (net 7))
   (segment (start 30.48 -48.006) (end 35.56 -48.006) (width 1) (layer "In2.Cu") (net 7))
@@
   (segment (start 40.259 -45.72) (end 40.005 -45.72) (width 0.5) (layer "B.Cu") (net 7))
   (segment (start 41.91 -10.922) (end 42.257 -11.269) (width 0.5) (layer "B.Cu") (net 7))
-  (segment (start 9.398 -42.483) (end 9.398 -43.434) (width 0.5) (layer "B.Cu") (net 7))
   (segment (start 38.155 -5.359) (end 38.155 -7.167) (width 0.5) (layer "B.Cu") (net 7))
   (segment (start 48.631999 -34.967999) (end 48.335 -34.671) (width 0.5) (layer "B.Cu") (net 7))
   (segment (start 24.167 -6.895) (end 24.558 -7.286) (width 0.5) (layer "B.Cu") (net 7))
+  (segment (start 9.652 -43.499) (end 9.652 -44.323) (width 0.5) (layer "B.Cu") (net 7))
   (segment (start 29.337 -4.699) (end 29.464 -4.572) (width 1) (layer "B.Cu") (net 7))
   (segment (start 29.337 -6.286) (end 29.337 -4.699) (width 1) (layer "B.Cu") (net 7))
@@
   (segment (start 44.196 -11.269) (end 44.196 -11.938) (width 1) (layer "B.Cu") (net 7))
   (segment (start 24.167 -5.406) (end 24.167 -6.895) (width 0.5) (layer "B.Cu") (net 7))
+  (segment (start 9.652 -44.323) (end 9.906 -44.577) (width 0.5) (layer "B.Cu") (net 7))
   (segment (start 44.196 -11.938) (end 46.228 -13.97) (width 1) (layer "B.Cu") (net 7))
-  (segment (start 9.398 -43.434) (end 9.652 -43.688) (width 0.5) (layer "B.Cu") (net 7))
   (segment (start 5.905 -28.575) (end 7.874 -28.575) (width 0.5) (layer "B.Cu") (net 8))
   (segment (start 20.955 -35.184) (end 21.6204 -35.184) (width 0.25) (layer "B.Cu") (net 9))
@@
   (segment (start 14.394 -32.954) (end 13.212 -32.954) (width 0.5) (layer "B.Cu") (net 66))
   (segment (start 7.295 -37.96) (end 7.93 -37.96) (width 0.5) (layer "B.Cu") (net 66))
-  (segment (start 9.398 -41.083) (end 9.398 -38.1) (width 0.5) (layer "B.Cu") (net 66))
   (segment (start 13.212 -32.954) (end 13.019 -33.147) (width 0.5) (layer "B.Cu") (net 66))
   (segment (start 9.258 -37.96) (end 9.398 -38.1) (width 0.5) (layer "B.Cu") (net 66))
   (segment (start 8.496 -33.16) (end 8.877 -33.16) (width 0.5) (layer "B.Cu") (net 66))
+  (segment (start 9.398 -39.178) (end 9.398 -38.1) (width 0.5) (layer "B.Cu") (net 66))
+  (via (at 12.64 -37.41) (size 0.8) (drill 0.4) (layers "F.Cu" "B.Cu") (net 67))
+  (via (at 10.4 -40.35) (size 0.8) (drill 0.4) (layers "F.Cu" "B.Cu") (net 67))
+  (segment (start 12.64 -38.11) (end 10.4 -40.35) (width 0.5) (layer "In2.Cu") (net 67))
+  (segment (start 12.64 -37.41) (end 12.64 -38.11) (width 0.5) (layer "In2.Cu") (net 67))
+  (segment (start 10.172 -40.578) (end 10.4 -40.35) (width 0.5) (layer "B.Cu") (net 67))
+  (segment (start 10.4 -40.35) (end 9.788 -40.962) (width 0.5) (layer "B.Cu") (net 67))
+  (segment (start 9.788 -40.962) (end 9.652 -40.962) (width 0.5) (layer "B.Cu") (net 67))
+  (segment (start 13.257 -37.41) (end 13.71 -36.957) (width 0.5) (layer "B.Cu") (net 67))
+  (segment (start 12.64 -37.41) (end 13.257 -37.41) (width 0.5) (layer "B.Cu") (net 67))
+  (segment (start 9.652 -40.832) (end 9.398 -40.578) (width 0.5) (layer "B.Cu") (net 67))
+  (segment (start 13.71 -37.598) (end 13.335 -37.973) (width 0.5) (layer "B.Cu") (net 67))
+  (segment (start 13.71 -37.725) (end 13.71 -36.957) (width 0.5) (layer "B.Cu") (net 67))
+  (segment (start 13.335 -37.973) (end 13.335 -37.332) (width 0.5) (layer "B.Cu") (net 67))
+  (segment (start 9.652 -42.099) (end 9.652 -40.962) (width 0.5) (layer "B.Cu") (net 67))
+  (segment (start 13.335 -37.332) (end 13.71 -36.957) (width 0.5) (layer "B.Cu") (net 67))
+  (segment (start 13.71 -36.957) (end 13.71 -37.598) (width 0.5) (layer "B.Cu") (net 67))
+  (segment (start 9.398 -40.578) (end 10.172 -40.578) (width 0.5) (layer "B.Cu") (net 67))
+  (segment (start 9.652 -40.962) (end 9.652 -40.832) (width 0.5) (layer "B.Cu") (net 67))
   (zone (net 1) (net_name "GND") (layer "F.Cu") (hatch edge 0.508)
     (connect_pads yes (clearance 0))

Commit message: Edit PCB
Other:
- rule pad_to_mask_clearance: 0 -> 0.2
Changed lines of the file:
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@@
       (dielectric_constraints no)
     )
-    (pad_to_mask_clearance 0)
+    (pad_to_mask_clearance 0.2)
     (pcbplotparams
       (layerselection 0x00010e0_ffffffff)

Commit message: Uprava projektovych dat
Parts:
- moved C13 173.9 mm to (156.5, 101.1)
- moved C3 173.9 mm to (141.1, 87.3)
- moved C9 173.9 mm to (159.7, 108.1)
- moved D4 173.9 mm to (168.6, 88.9)
- moved D5 173.9 mm to (168.6, 92.3)
- moved D6 173.9 mm to (168.6, 95.8)
- moved D7 173.9 mm to (168.6, 85.4)
- moved D9 173.9 mm to (132.0, 80.8)
- moved FL1 173.9 mm to (147.6, 110.8)
- moved L1 173.9 mm to (137.4, 86.6)
- moved L2 173.9 mm to (157.2, 104.1)
- moved M2 173.9 mm to (127.7, 118.2)
- moved M4 173.9 mm to (167.7, 118.2)
- moved Q3 173.9 mm to (162.7, 82.5)
- moved R13 173.9 mm to (155.4, 81.9)
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