File: hw/sch_pcb/TFGPS01B.kicad_sch (KiCad schematic)
At the start: 71 parts, among them J1 SM10B-GHS-TB, J2 USBC_USB4105-GF-A, J3 SM06B-GHS-TB, J4 SM04B-GHS-TB, J5 SM08B-GHS-TB, M1 HOLE, M2 HOLE, M3 HOLE, M4 HOLE, Q1 BC817-25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

Commit message: #22
Parts:
- added R?: 10k, Mlab_R:SMD-0805, symbol Device:R
- R28: value 100R -> 20k; UST_ID 5c70984512875079b91f8977 -> 5c70984612875079b91f89a3
Connections:
- net SAFETY_SW_LED: now also R?.1
- net SAFE_VCC: now also R?.2
Changed lines of the file:
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@@
-(kicad_sch (version 20210126) (generator eeschema)
+(kicad_sch (version 20210406) (generator eeschema)
   (paper "A4")
   (title_block
@@
   (junction (at 125.73 38.1) (diameter 1.016) (color 0 0 0 0))
   (junction (at 128.27 58.42) (diameter 1.016) (color 0 0 0 0))
+  (junction (at 152.4 45.72) (diameter 1.016) (color 0 0 0 0))
   (junction (at 170.18 39.37) (diameter 1.016) (color 0 0 0 0))
   (junction (at 181.61 74.93) (diameter 1.016) (color 0 0 0 0))
@@
     (stroke (width 0) (type solid) (color 0 0 0 0))
   )
-  (wire (pts (xy 151.13 45.72) (xy 153.67 45.72))
+  (wire (pts (xy 151.13 45.72) (xy 152.4 45.72))
     (stroke (width 0) (type solid) (color 0 0 0 0))
   )
@@
     (stroke (width 0) (type solid) (color 0 0 0 0))
   )
+  (wire (pts (xy 152.4 31.75) (xy 152.4 33.655))
+    (stroke (width 0) (type solid) (color 0 0 0 0))
+  )
+  (wire (pts (xy 152.4 41.275) (xy 152.4 45.72))
+    (stroke (width 0) (type solid) (color 0 0 0 0))
+  )
+  (wire (pts (xy 152.4 45.72) (xy 153.67 45.72))
+    (stroke (width 0) (type solid) (color 0 0 0 0))
+  )
   (wire (pts (xy 160.02 109.22) (xy 160.02 114.3))
     (stroke (width 0) (type solid) (color 0 0 0 0))
@@
     (effects (font (size 1.524 1.524)) (justify right bottom))
   )
+  (label "SAFE_VCC" (at 152.4 31.75 0)
+    (effects (font (size 1.524 1.524)) (justify left bottom))
+  )
   (label "ARM" (at 185.42 39.37 180)
     (effects (font (size 1.524 1.524)) (justify right bottom))
@@
     (pin "2")
   )
+  (symbol (lib_id "Device:R") (at 152.4 37.465 180) (unit 1)
+    (in_bom yes) (on_board yes)
+    (property "Reference" "R?" (id 0) (at 149.7138 38.735 90))
+    (property "Value" "10k" (id 1) (at 154.553 37.465 90))
+    (property "Footprint" "Mlab_R:SMD-0805" (id 2) (at 154.178 37.465 90)
+      (effects (font (size 1.27 1.27)) hide)
+    )
+    (property "Datasheet" "~" (id 3) (at 152.4 37.465 0)
+      (effects (font (size 1.27 1.27)) hide)
+    )
+    (property "UST_ID" "" (id 4) (at 152.4 37.465 0)
+      (effects (font (size 1.27 1.27)) hide)
+    )
+    (pin "1")
+    (pin "2")
+  )
   (symbol (lib_id "Device:R") (at 157.48 45.72 90) (unit 1)
     (in_bom yes) (on_board yes)
     (property "Reference" "R28" (id 0) (at 156.21 43.0338 90))
-    (property "Value" "100R" (id 1) (at 157.48 47.873 90))
+    (property "Value" "20k" (id 1) (at 157.48 47.873 90))
     (property "Footprint" "Mlab_R:SMD-0805" (id 2) (at 157.48 47.498 90)
       (effects (font (size 1.27 1.27)) hide)
@@
       (effects (font (size 1.27 1.27)) hide)
     )
-    (property "UST_ID" "5c70984512875079b91f8977" (id 4) (at 157.48 45.72 0)
+    (property "UST_ID" "5c70984612875079b91f89a3" (id 4) (at 157.48 45.72 0)
       (effects (font (size 1.27 1.27)) hide)
     )
@@
     )
     (path "/d6a4e04e-8df6-4986-9125-2e4dff9106e1"
-      (reference "R28") (unit 1) (value "100R") (footprint "Mlab_R:SMD-0805")
+      (reference "R28") (unit 1) (value "20k") (footprint "Mlab_R:SMD-0805")
+    )
+    (path "/2895353c-22c9-4754-9433-fb9ee36359e3"
+      (reference "R?") (unit 1) (value "10k") (footprint "Mlab_R:SMD-0805")
     )
     (path "/00000000-0000-0000-0000-00005e8337ab"

Commit message: Edit schema
Parts:
- C13: value 1pF -> 1p5F; UST_ID 5c70984712875079b91f8b26 -> (none)
- L2: value 4n7H -> 5n6H; UST_ID 5fa100d812875025b39779cf -> (none)
- R13: value 100R -> 10k; UST_ID 5c70984512875079b91f8977 -> (none)
- U4: value MAX2656 -> MAX2655
- gave numbers to parts that had none: 1
Changed lines of the file:
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@@
     (in_bom yes) (on_board yes)
     (property "Reference" "L2" (id 0) (at 250.19 94.3418 90))
-    (property "Value" "4n7H" (id 1) (at 250.19 96.64 90))
+    (property "Value" "5n6H" (id 1) (at 250.19 96.64 90))
     (property "Footprint" "Mlab_R:SMD-0805" (id 2) (at 250.19 99.06 0)
       (effects (font (size 1.27 1.27)) hide)
@@
       (effects (font (size 1.27 1.27)) hide)
     )
-    (property "UST_ID" "5fa100d812875025b39779cf" (id 4) (at 250.19 99.06 0)
+    (property "UST_ID" "" (id 4) (at 250.19 99.06 0)
       (effects (font (size 1.27 1.27)) hide)
     )
@@
     (in_bom yes) (on_board yes)
     (property "Reference" "R13" (id 0) (at 127 177.6538 90))
-    (property "Value" "100R" (id 1) (at 128.27 182.493 90))
+    (property "Value" "10k" (id 1) (at 128.27 182.493 90))
     (property "Footprint" "Mlab_R:SMD-0805" (id 2) (at 128.27 182.118 90)
       (effects (font (size 1.27 1.27)) hide)
@@
       (effects (font (size 1.27 1.27)) hide)
     )
-    (property "UST_ID" "5c70984512875079b91f8977" (id 4) (at 128.27 180.34 0)
+    (property "UST_ID" "" (id 4) (at 128.27 180.34 0)
       (effects (font (size 1.27 1.27)) hide)
     )
@@
   (symbol (lib_id "Device:R") (at 152.4 37.465 180) (unit 1)
     (in_bom yes) (on_board yes)
-    (property "Reference" "R?" (id 0) (at 149.7138 38.735 90))
+    (property "Reference" "R25" (id 0) (at 149.7138 38.735 90))
     (property "Value" "10k" (id 1) (at 154.553 37.465 90))
     (property "Footprint" "Mlab_R:SMD-0805" (id 2) (at 154.178 37.465 90)
@@
       (effects (font (size 1.27 1.27)) (justify right))
     )
-    (property "Value" "1pF" (id 1) (at 259.461 106.559 0)
+    (property "Value" "1p5F" (id 1) (at 259.461 106.559 0)
       (effects (font (size 1.27 1.27)) (justify right))
     )
@@
       (effects (font (size 1.27 1.27)) hide)
     )
-    (property "UST_ID" "5c70984712875079b91f8b26" (id 4) (at 256.54 105.41 0)
+    (property "UST_ID" "" (id 4) (at 256.54 105.41 0)
       (effects (font (size 1.27 1.27)) hide)
     )
@@
       (effects (font (size 1.27 1.27)) (justify right))
     )
-    (property "Value" "MAX2656" (id 1) (at 233.4261 91.9543 0)
+    (property "Value" "MAX2655" (id 1) (at 233.4261 91.9543 0)
       (effects (font (size 1.27 1.27)) (justify right))
     )
@@
     )
     (path "/86deb435-ac6f-4922-806a-0998ac1a3708"
-      (reference "C13") (unit 1) (value "1pF") (footprint "Mlab_R:SMD-0805")
+      (reference "C13") (unit 1) (value "1p5F") (footprint "Mlab_R:SMD-0805")
     )
     (path "/b830f0d4-d797-4b91-b70b-9b3a7a4c51f0"
@@
     )
     (path "/4df28642-4338-4e55-b154-9d794c85815c"
-      (reference "L2") (unit 1) (value "4n7H") (footprint "Mlab_R:SMD-0805")
+      (reference "L2") (unit 1) (value "5n6H") (footprint "Mlab_R:SMD-0805")
     )
     (path "/00000000-0000-0000-0000-0000549d7549"
@@
     )
     (path "/cdd98aa8-39c3-4902-a0e7-b4479d95ffc5"
-      (reference "R13") (unit 1) (value "100R") (footprint "Mlab_R:SMD-0805")
+      (reference "R13") (unit 1) (value "10k") (footprint "Mlab_R:SMD-0805")
     )
     (path "/7b4cb5de-acfc-4eb8-b423-1fe9cedbdaaf"
@@
       (reference "R24") (unit 1) (value "220R") (footprint "Mlab_R:SMD-0805")
     )
+    (path "/2895353c-22c9-4754-9433-fb9ee36359e3"
+      (reference "R25") (unit 1) (value "10k") (footprint "Mlab_R:SMD-0805")
+    )
     (path "/d1585a21-b520-4562-97dd-1e6ebc7a6516"
       (reference "R26") (unit 1) (value "12k") (footprint "Mlab_R:SMD-0805")
@@
       (reference "R28") (unit 1) (value "20k") (footprint "Mlab_R:SMD-0805")
     )
-    (path "/2895353c-22c9-4754-9433-fb9ee36359e3"
-      (reference "R?") (unit 1) (value "10k") (footprint "Mlab_R:SMD-0805")
-    )
     (path "/00000000-0000-0000-0000-00005e8337ab"
       (reference "U1") (unit 1) (value "MIC5504-3.3YM5") (footprint "Package_TO_SOT_SMD:SOT-23-5")
@@
     )
     (path "/e9490243-5a68-4bbb-a1d9-29a68cf133c8"
-      (reference "U4") (unit 1) (value "MAX2656") (footprint "Package_TO_SOT_SMD:SOT-363_SC-70-6")
-    )
-  )
+      (reference "U4") (unit 1) (value "MAX2655") (footprint "Package_TO_SOT_SMD:SOT-363_SC-70-6")
+    )
+  )

Commit message: Edit schema
Parts:
- added D9: 15MQ040N, Diode_SMD:D_SMA, symbol Device:D
- added F1: 750mA, Fuse:Fuse_0805_2012Metric, symbol Device:Fuse
Connections:
- net +5V: now also D9.1 (K); no longer J2.A4/B9 (VBUS), J2.B4/A9 (VBUS), U2.5 (VBUS)
- new net: D9.2 (A), F1.2
- new net VBUS: F1.1, J2.A4/B9 (VBUS), J2.B4/A9 (VBUS), U2.5 (VBUS)
Other:
- moved on the sheet: C3, C4, C5, D2, D3, D4, L1, Q1, R13, R19, R4, U1

Commit message: Edit SCH
Parts:
- removed F1: 750mA, Fuse:Fuse_0805_2012Metric, symbol Device:Fuse
- added D10: 15MQ040N, Diode_SMD:D_SMA, symbol Device:D
Connections:
- net +5V: now also D10.2 (A); no longer D2.1 (K), D9.1 (K), L1.1
- net VBUS: now also D9.2 (A)
- new net: D10.1 (K), D2.1 (K), D9.1 (K), L1.1
Changed lines of the file:
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@@
     (stroke (width 0) (type solid) (color 0 0 0 0))
   )
-  (wire (pts (xy 28.575 170.815) (xy 30.48 170.815))
-    (stroke (width 0) (type solid) (color 0 0 0 0))
-  )
   (wire (pts (xy 29.21 21.59) (xy 29.21 19.05))
     (stroke (width 0) (type solid) (color 0 0 0 0))
@@
     (stroke (width 0) (type solid) (color 0 0 0 0))
   )
-  (wire (pts (xy 38.1 170.815) (xy 39.37 170.815))
+  (wire (pts (xy 36.195 170.815) (xy 39.37 170.815))
     (stroke (width 0) (type solid) (color 0 0 0 0))
   )
@@
     (stroke (width 0) (type solid) (color 0 0 0 0))
   )
+  (wire (pts (xy 54.61 156.845) (xy 54.61 158.115))
+    (stroke (width 0) (type solid) (color 0 0 0 0))
+  )
   (wire (pts (xy 54.61 165.735) (xy 54.61 170.815))
     (stroke (width 0) (type solid) (color 0 0 0 0))
@@
     (effects (font (size 1.524 1.524)) (justify left bottom))
   )
-  (label "VBUS" (at 28.575 170.815 180)
-    (effects (font (size 1.524 1.524)) (justify right bottom))
-  )
   (label "RX" (at 29.21 24.13 0)
     (effects (font (size 1.524 1.524)) (justify left bottom))
@@
     (effects (font (size 1.524 1.524)) (justify left bottom))
   )
+  (label "VBUS" (at 36.195 170.815 180)
+    (effects (font (size 1.524 1.524)) (justify right bottom))
+  )
   (label "VBUS" (at 44.45 64.77 0)
     (effects (font (size 1.524 1.524)) (justify left bottom))
@@
     (pin "1")
   )
-  (symbol (lib_id "power:+5V") (at 54.61 165.735 0) (unit 1)
+  (symbol (lib_id "power:+5V") (at 54.61 156.845 0) (unit 1)
     (in_bom yes) (on_board yes)
-    (property "Reference" "#PWR04" (id 0) (at 54.61 169.545 0)
+    (property "Reference" "#PWR04" (id 0) (at 54.61 160.655 0)
       (effects (font (size 1.27 1.27)) hide)
     )
-    (property "Value" "+5V" (id 1) (at 54.9783 161.4106 0))
-    (property "Footprint" "" (id 2) (at 54.61 165.735 0)
+    (property "Value" "+5V" (id 1) (at 54.9783 152.5206 0))
+    (property "Footprint" "" (id 2) (at 54.61 156.845 0)
       (effects (font (size 1.27 1.27)) hide)
     )
-    (property "Datasheet" "" (id 3) (at 54.61 165.735 0)
+    (property "Datasheet" "" (id 3) (at 54.61 156.845 0)
       (effects (font (size 1.27 1.27)) hide)
     )
@@
     (pin "2")
   )
-  (symbol (lib_id "Device:Fuse") (at 34.29 170.815 90) (unit 1)
-    (in_bom yes) (on_board yes) (fields_autoplaced)
-    (property "Reference" "F1" (id 0) (at 34.29 166.6198 90))
-    (property "Value" "750mA" (id 1) (at 34.29 168.9185 90))
-    (property "Footprint" "Fuse:Fuse_0805_2012Metric" (id 2) (at 34.29 172.593 90)
-      (effects (font (size 1.27 1.27)) hide)
-    )
-    (property "Datasheet" "5c70984512875079b91f88d4" (id 3) (at 34.29 170.815 0)
-      (effects (font (size 1.27 1.27)) hide)
-    )
-    (pin "1")
-    (pin "2")
-  )
   (symbol (lib_id "Device:R") (at 19.05 127 0) (unit 1)
     (in_bom yes) (on_board yes)
@@
     (pin "2")
   )
+  (symbol (lib_id "Device:D") (at 54.61 161.925 90) (unit 1)
+    (in_bom yes) (on_board yes)
+    (property "Reference" "D10" (id 0) (at 52.6034 163.0934 90)
+      (effects (font (size 1.27 1.27)) (justify left))
+    )
+    (property "Value" "15MQ040N" (id 1) (at 52.6034 160.782 90)
+      (effects (font (size 1.27 1.27)) (justify left))
+    )
+    (property "Footprint" "Diode_SMD:D_SMA" (id 2) (at 54.61 161.925 0)
+      (effects (font (size 1.27 1.27)) hide)
+    )
+    (property "Datasheet" "~" (id 3) (at 54.61 161.925 0)
+      (effects (font (size 1.27 1.27)) hide)
+    )
+    (property "UST_ID" "5c70984512875079b91f88b0" (id 4) (at 54.61 161.925 0)
+      (effects (font (size 1.27 1.27)) hide)
+    )
+    (pin "1")
+    (pin "2")
+  )
   (symbol (lib_id "Device:D") (at 54.61 177.165 270) (unit 1)
     (in_bom yes) (on_board yes)
@@
       (reference "D9") (unit 1) (value "15MQ040N") (footprint "Diode_SMD:D_SMA")
     )
-    (path "/757879af-e6f3-4f64-afa4-29c9cf356a0a"
-      (reference "F1") (unit 1) (value "750mA") (footprint "Fuse:Fuse_0805_2012Metric")
+    (path "/73793ff1-347e-42b9-88d0-c9a8ffebabe7"
+      (reference "D10") (unit 1) (value "15MQ040N") (footprint "Diode_SMD:D_SMA")
     )
     (path "/e78163e9-482e-4227-9608-722196227914"

Commit message: Edit SCH
Parts:
- removed D10, D9: 15MQ040N, Diode_SMD:D_SMA, symbol Device:D
- added D10, D9: BZX585-B5V6.115, Diode_SMD:D_SOD-523, symbol MLAB_D:D_ZENER
Connections:
- net +5V: now also D2.1 (K), D9.2 (A)
- net VBUS: now also D10.2 (A)
- net at L1.1: now also D10.1 (K), D9.1 (K); no longer D2.1 (K)
Other:
- moved on the sheet: D2

Commit message: Edit PCB
Parts:
- C13: UST_ID (none) -> 60d587411287500165f85b5f
- L2: UST_ID (none) -> 5c70984412875079b91f8803
- R13, R25: UST_ID (none) -> 5c70984612875079b91f899f
Changed lines of the file:
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@@
       (effects (font (size 1.27 1.27)) hide)
     )
-    (property "UST_ID" "" (id 4) (at 250.19 99.06 0)
+    (property "UST_ID" "5c70984412875079b91f8803" (id 4) (at 250.19 99.06 0)
       (effects (font (size 1.27 1.27)) hide)
     )
@@
       (effects (font (size 1.27 1.27)) hide)
     )
-    (property "UST_ID" "" (id 4) (at 144.78 180.34 0)
+    (property "UST_ID" "5c70984612875079b91f899f" (id 4) (at 144.78 180.34 0)
       (effects (font (size 1.27 1.27)) hide)
     )
@@
       (effects (font (size 1.27 1.27)) hide)
     )
-    (property "UST_ID" "" (id 4) (at 152.4 37.465 0)
+    (property "UST_ID" "5c70984612875079b91f899f" (id 4) (at 152.4 37.465 0)
       (effects (font (size 1.27 1.27)) hide)
     )
@@
       (effects (font (size 1.27 1.27)) hide)
     )
-    (property "UST_ID" "" (id 4) (at 256.54 105.41 0)
-      (effects (font (size 1.27 1.27)) hide)
-    )
+    (property "UST_ID" "60d587411287500165f85b5f" (id 4) (at 256.54 105.41 0)
+      (effects (font (size 1.27 1.27)) hide)
+    )
